Commit message: Add rack grasp and place

File: src/ndf_robot/descriptions/hanging/table/table_shelf.urdf (robot description, URDF)
Before this commit: robot table.urdf, 2 links, 1 joints
Links:
- link shelf: geometry collision mesh filename=shelf_back.stl scale=1.0 1.0 1.0; visual mesh filename=shelf_back.stl scale=1.0 1.0 1.0

File: src/ndf_robot/descriptions/hanging/table/table_shelf_old.urdf (robot description, URDF)
Before this commit: robot table.urdf, 2 links, 1 joints
Links:
- removed link rack
- added link shelf; collision mesh filename=shelf_back.stl scale=1.0 0.75 0.5; visual mesh filename=shelf_back.stl scale=0.75 0.75 0.5
Joints:
- removed joint table2rack
- added joint table2shelf: type fixed, parent baseLink, child shelf, origin xyz=-0.5 0.125 0.625 rpy=0 0 -1.57
