Commit message: Refine simulation

File: src/ndf_robot/descriptions/hanging/table/table_rack_tmp.urdf (robot description, URDF)
Before this commit: robot table.urdf, 2 links, 1 joints
Links:
- removed link rack
Joints:
- removed joint table2rack

Commit message: Add cylinder query points

File: src/ndf_robot/descriptions/hanging/table/table_rack_tmp.urdf (robot description, URDF)
Before this commit: robot table.urdf, 1 links, 0 joints
Links:
- added link rack; collision mesh filename=simple_rack.obj scale=1.0 1.0 1.0; visual mesh filename=simple_rack.obj scale=1.0 1.0 1.0
Joints:
- added joint table2rack: type fixed, parent baseLink, child rack, origin xyz=0.3 -0.1 0.635 rpy=0 0 3.1415

Commit message: Add preliminary shelf teleport

File: src/ndf_robot/descriptions/hanging/table/table_rack_tmp.urdf (robot description, URDF)
Before this commit: robot table.urdf, 2 links, 1 joints
Links:
- removed link rack
- added link shelf; collision mesh filename=shelf_back.stl scale=0.75 0.75 0.5; visual mesh filename=shelf_back.stl scale=0.75 0.75 0.5
Joints:
- removed joint table2rack
- added joint table2shelf: type fixed, parent baseLink, child shelf, origin xyz=-0.5 0.125 0.625 rpy=0 0 -1.57

Commit message: Add option to save best opt or all opt

File: src/ndf_robot/descriptions/hanging/table/table_rack_tmp.urdf (robot description, URDF)
Before this commit: robot table.urdf, 1 links, 0 joints
Links:
- added link shelf; collision mesh filename=shelf_back.stl scale=0.75 0.75 0.5; visual mesh filename=shelf_back.stl scale=0.75 0.75 0.5
Joints:
- added joint table2shelf: type fixed, parent baseLink, child shelf, origin xyz=-0.5 0.125 0.625 rpy=0 0 -1.57

Commit message: remove collisions before preplace

File: src/ndf_robot/descriptions/hanging/table/table_rack_tmp.urdf (robot description, URDF)
Before this commit: robot table.urdf, 2 links, 1 joints
Links:
- removed link shelf
- added link rack; collision mesh filename=simple_rack.obj scale=1.0 1.0 1.0; visual mesh filename=simple_rack.obj scale=1.0 1.0 1.0
Joints:
- removed joint table2shelf
- added joint table2rack: type fixed, parent baseLink, child rack, origin xyz=0.3 -0.1 0.635 rpy=0 0 3.1415

Commit message: Debug bottle grasp

File: src/ndf_robot/descriptions/hanging/table/table_rack_tmp.urdf (robot description, URDF)
Before this commit: robot table.urdf, 2 links, 1 joints
Links:
- removed link rack
- added link shelf; collision mesh filename=shelf_back.stl scale=1.0 0.75 0.5; visual mesh filename=shelf_back.stl scale=0.75 0.75 0.5
Joints:
- removed joint table2rack
- added joint table2shelf: type fixed, parent baseLink, child shelf, origin xyz=-0.5 0.125 0.625 rpy=0 0 -1.57

Commit message: Tune shelf place

File: src/ndf_robot/descriptions/hanging/table/table_rack_tmp.urdf (robot description, URDF)
Before this commit: robot table.urdf, 2 links, 1 joints
Links:
- removed link rack
- added link shelf; collision mesh filename=shelf_back.stl scale=1.0 0.75 0.5; visual mesh filename=shelf_back.stl scale=0.75 0.75 0.5
Joints:
- removed joint table2rack
- added joint table2shelf: type fixed, parent baseLink, child shelf, origin xyz=-0.5 0.125 0.625 rpy=0 0 -1.57

File: src/ndf_robot/descriptions/hanging/table/table_shelf.urdf (robot description, URDF)
Before this commit: robot table.urdf, 2 links, 1 joints
Links:
- link shelf: geometry collision mesh filename=shelf_back.stl scale=1.0 0.75 0.5; visual mesh filename=shelf_back.stl scale=0.75 0.75 0.5

Commit message: Misc updates and change readme

File: src/ndf_robot/descriptions/hanging/table/table_rack_tmp.urdf (robot description, URDF)
Before this commit: robot table.urdf, 2 links, 1 joints
Links:
- removed link shelf
Joints:
- removed joint table2shelf

Commit message: Debug geom optimizer transform, run geom trials

File: src/ndf_robot/descriptions/hanging/table/table_rack_tmp.urdf (robot description, URDF)
Before this commit: robot table.urdf, 1 links, 0 joints
Links:
- added link shelf; collision mesh filename=shelf_back.stl scale=1.0 0.75 0.5; visual mesh filename=shelf_back.stl scale=0.75 0.75 0.5
Joints:
- added joint table2shelf: type fixed, parent baseLink, child shelf, origin xyz=-0.5 0.125 0.625 rpy=0 0 -1.57
